Commit message: commit

File: src/jetson_nano_bot/launch_jetson_nano_bot/urdf/my_robot_base.xacro (robot description, xacro)
@@ -28,5 +28,5 @@
     <parent link="base_link"/>
     <child link="laser"/>
-    <origin xyz="0 0 0.2" rpy="0 0 3.141592"/>
+    <origin xyz="0 0 0.2" rpy="0 0 0"/>
     <!--<axis xyz="0 1 0"/>-->
   </joint>
